File: mini_project_one/kicad/kicad_model/mp1.kicad_pcb (KiCad board)
At the start: 2 copper layers, 17.3 x 13.6 mm, 17 parts, among them J1 48037-0001, U1 MCP1702T-3302E/CB, U2 MCP6022T-I/ST

Commit message: added gitignore and updated parts libraries
Parts:
- D1: footprint LTST-C170TBKT:DIOC200X125X110 -> 160-1579-1-ND:160-1579-1-ND
- U1: footprint MCP1702T:MCP1702T-3302E&slash_CB -> MCP1702T-3302E-CBCT-ND:MCP1702T-3302E&slash_CB
- U2: footprint MCP6022T:MCP6022T-I&slash_ST -> MCP6022T-I-STCT-ND:MCP6022T-I&slash_ST

Commit message: updated design and added bom
Parts:
- removed the C2 at (99.6, 81.5)
- moved C3 5.90 mm to (96.3, 84.3), turned to -90 degrees
- moved R5 5.88 mm to (104.3, 78.7)
- moved C4 3.65 mm to (99.7, 81.6), turned to 180 degrees
- moved R4 2.91 mm to (100.1, 87.6), turned to -90 degrees
- moved U1 2.84 mm to (98.3, 78.3)
- moved R1 2.79 mm to (102.8, 78.7)
- moved R7 2.78 mm to (98.6, 87.6), turned to -90 degrees
- moved C2 2.74 mm to (101.3, 78.7)
- moved C1 2.29 mm to (96.4, 81.0)
- moved R6 1.81 mm to (103.2, 87.6), turned to -90 degrees
- moved R3 1.34 mm to (101.7, 87.6), turned to -90 degrees
- moved D1 1.28 mm to (96.7, 87.8), turned to 90 degrees
- moved R8 0.92 mm to (104.7, 87.6), turned to -90 degrees
- moved U2 0.10 mm to (101.1, 84.1)
- renumbered C3 to C2, C4 to C3, C5 to C4
Routing:
- net Net-(C2-Pad1): track 21.6 -> 14.1 mm
- net Net-(C4-Pad2): track 9.08 -> 15.9 mm, vias 2 -> 0
- net Net-(R5-Pad2): track 3.66 -> 10.2 mm
- net Net-(R5-Pad1): track 4.31 -> 9.13 mm
- net Net-(R4-Pad2): track 15.1 -> 10.4 mm
- net Net-(C1-Pad1): track 17.3 -> 13.6 mm
- net GND: track 37.5 -> 34.1 mm, vias 3 -> 1
- net Net-(R3-Pad1): track 6.43 -> 3.58 mm
- net Net-(R3-Pad2): track 9.96 -> 7.77 mm, vias 0 -> 2
- net Net-(D1-Pad+): track 1.58 -> 3.17 mm
Other:
- board size 17.3 x 13.6 mm -> 16.7 x 13.6 mm
