File: mini_project_one/kicad/kicad_model/mp1.kicad_sch (KiCad schematic)
At the start: 17 parts, among them J1 48037-0001, U1 MCP1702T-3302E/CB, U2 MCP6022T-I/ST

Commit message: added gitignore and updated parts libraries
Parts:
- removed J1: 48037-0001, 48037-0001:MOLEX_48037-0001, symbol WM17117-ND:48037-0001
- removed U1: MCP1702T-3302E/CB, MCP1702T:MCP1702T-3302E&slash_CB, symbol MCP1702T-3302E:MCP1702T-3302E/CB
- removed U2: MCP6022T-I/ST, MCP6022T:MCP6022T-I&slash_ST, symbol MCP6022T-I/STCT-ND:MCP6022T-I/ST
- added J1: 48037-0001, 48037-0001:MOLEX_48037-0001, symbol 48037-0001:48037-0001
- added U1: MCP1702T-3302E/CB, MCP1702T-3302E-CBCT-ND:MCP1702T-3302E&slash_CB, symbol MCP1702T-3302E-CBCT-ND:MCP1702T-3302E/CB
- added U2: MCP6022T-I/ST, MCP6022T-I-STCT-ND:MCP6022T-I&slash_ST, symbol MCP6022T-I-STCT-ND:MCP6022T-I/ST
- D1: footprint LTST-C170TBKT:DIOC200X125X110 -> 160-1579-1-ND:160-1579-1-ND
Connections:
- net GND: now also J1.4 (GND), J1.S1 (SHIELD), J1.S2 (SHIELD), U1.1 (GND), U2.4 (VSS)
- net at R3.1: now also U2.1 (VOUTA), U2.2 (VINA-)
- net at R1.1, R2.2: now also U2.3 (VINA+)
- net at R3.2, R4.1: now also U2.5 (VINB+)
- net at C5.2, R8.2: now also U2.6 (VINB-)
- net at R4.2, R6.2, R7.1: now also U2.7 (VOUTB)
- net at C2.1, C3.1, C4.1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: now also U1.2 (VOUT), U2.8 (VDD)
- net at C1.1: now also J1.1 (VCC), U1.3 (VIN)
Other:
- moved on the sheet: C1, C5

Commit message: updated design and added bom
Parts:
- removed C2: 1U, Capacitor_SMD:C_0603_1608Metric_Pad1.08x0.95mm_HandSolder, symbol Device:C
- renumbered C3 to C2, C4 to C3, C5 to C4
Other:
- moved on the sheet: D1
Changed lines of the file:
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@@
   (junction (at 74.93 99.06) (diameter 0) (color 0 0 0 0)
   )
-  (junction (at 123.19 106.68) (diameter 0) (color 0 0 0 0)
-  )
   (junction (at 130.81 86.36) (diameter 0) (color 0 0 0 0)
   )
@@
   )
   (junction (at 80.01 99.06) (diameter 0) (color 0 0 0 0)
-  )
-  (junction (at 123.19 86.36) (diameter 0) (color 0 0 0 0)
   )
   (junction (at 208.28 88.9) (diameter 0) (color 0 0 0 0)
@@
     (stroke (width 0) (type default) (color 0 0 0 0))
   )
-  (wire (pts (xy 123.19 106.68) (xy 132.08 106.68))
+  (wire (pts (xy 102.87 106.68) (xy 132.08 106.68))
     (stroke (width 0) (type default) (color 0 0 0 0))
   )
@@
     (stroke (width 0) (type default) (color 0 0 0 0))
   )
-  (wire (pts (xy 102.87 106.68) (xy 123.19 106.68))
-    (stroke (width 0) (type default) (color 0 0 0 0))
-  )
   (wire (pts (xy 69.85 93.98) (xy 74.93 93.98))
     (stroke (width 0) (type default) (color 0 0 0 0))
@@
     (stroke (width 0) (type default) (color 0 0 0 0))
   )
-  (wire (pts (xy 123.19 93.98) (xy 123.19 106.68))
-    (stroke (width 0) (type default) (color 0 0 0 0))
-  )
   (wire (pts (xy 140.97 86.36) (xy 143.51 86.36))
     (stroke (width 0) (type default) (color 0 0 0 0))
@@
     (stroke (width 0) (type default) (color 0 0 0 0))
   )
-  (symbol (lib_id "160-1579-1-ND:LTST-C170TBKT") (at 227.33 106.68 90) (unit 1)
-    (in_bom yes) (on_board yes) (fields_autoplaced)
-    (property "Reference" "D1" (id 0) (at 229.87 104.4955 90)
-      (effects (font (size 1.27 1.27)) (justify right))
-    )
-    (property "Value" "LTST-C170TBKT" (id 1) (at 229.87 107.0355 90)
-      (effects (font (size 1.27 1.27)) (justify right))
+  (symbol (lib_id "160-1579-1-ND:LTST-C170TBKT") (at 227.33 106.68 270) (mirror x) (unit 1)
+    (in_bom yes) (on_board yes) (fields_autoplaced)
+    (property "Reference" "D1" (id 0) (at 232.41 104.4955 90)
+      (effects (font (size 1.27 1.27)) (justify left))
+    )
+    (property "Value" "LTST-C170TBKT" (id 1) (at 232.41 107.0355 90)
+      (effects (font (size 1.27 1.27)) (justify left))
     )
     (property "Footprint" "160-1579-1-ND:160-1579-1-ND" (id 2) (at 227.33 106.68 0)
@@
   (symbol (lib_id "Device:C") (at 132.08 102.87 0) (unit 1)
     (in_bom yes) (on_board yes)
-    (property "Reference" "C3" (id 0) (at 127 101.6 0)
+    (property "Reference" "C2" (id 0) (at 127 101.6 0)
       (effects (font (size 1.27 1.27)) (justify left))
     )
@@
     (pin "2")
   )
-  (symbol (lib_id "Device:C") (at 123.19 90.17 0) (unit 1)
-    (in_bom yes) (on_board yes) (fields_autoplaced)
-    (property "Reference" "C2" (id 0) (at 127 88.8999 0)
-      (effects (font (size 1.27 1.27)) (justify left))
-    )
-    (property "Value" "1U" (id 1) (at 127 91.4399 0)
-      (effects (font (size 1.27 1.27)) (justify left))
-    )
-    (property "Footprint" "Capacitor_SMD:C_0603_1608Metric_Pad1.08x0.95mm_HandSolder" (id 2) (at 124.1552 93.98 0)
-      (effects (font (size 1.27 1.27)) hide)
-    )
-    (property "Datasheet" "~" (id 3) (at 123.19 90.17 0)
-      (effects (font (size 1.27 1.27)) hide)
-    )
-    (pin "1")
-    (pin "2")
-  )
   (symbol (lib_id "MCP1702T-3302E-CBCT-ND:MCP1702T-3302E{slash}CB") (at 82.55 88.9 0) (unit 1)
     (in_bom yes) (on_board yes) (fields_autoplaced)
@@
   (symbol (lib_id "Device:C") (at 193.04 106.68 180) (unit 1)
     (in_bom yes) (on_board yes)
-    (property "Reference" "C5" (id 0) (at 196.85 105.41 0)
+    (property "Reference" "C4" (id 0) (at 196.85 105.41 0)
       (effects (font (size 1.27 1.27)) (justify right))
     )
@@
   (symbol (lib_id "Device:C") (at 140.97 102.87 0) (mirror y) (unit 1)
     (in_bom yes) (on_board yes)
-    (property "Reference" "C4" (id 0) (at 146.05 101.6 0)
+    (property "Reference" "C3" (id 0) (at 146.05 101.6 0)
       (effects (font (size 1.27 1.27)) (justify left))
     )
@@
       (reference "C1") (unit 1) (value "1U") (footprint "Capacitor_SMD:C_0603_1608Metric_Pad1.08x0.95mm_HandSolder")
     )
-    (path "/7e913f02-9af5-4e50-b678-2080dc06157c"
+    (path "/563078bb-97d4-437e-9842-7ccf8494b9c7"
       (reference "C2") (unit 1) (value "1U") (footprint "Capacitor_SMD:C_0603_1608Metric_Pad1.08x0.95mm_HandSolder")
     )
-    (path "/563078bb-97d4-437e-9842-7ccf8494b9c7"
-      (reference "C3") (unit 1) (value "1U") (footprint "Capacitor_SMD:C_0603_1608Metric_Pad1.08x0.95mm_HandSolder")
-    )
     (path "/e3153f3e-e860-4db0-9737-5eb20caf724d"
+      (reference "C3") (unit 1) (value ".1U") (footprint "Capacitor_SMD:C_0603_1608Metric_Pad1.08x0.95mm_HandSolder")
+    )
+    (path "/bc6f3101-5000-4fd2-8fa2-f9d28dcd8b01"
       (reference "C4") (unit 1) (value ".1U") (footprint "Capacitor_SMD:C_0603_1608Metric_Pad1.08x0.95mm_HandSolder")
     )
-    (path "/bc6f3101-5000-4fd2-8fa2-f9d28dcd8b01"
-      (reference "C5") (unit 1) (value ".1U") (footprint "Capacitor_SMD:C_0603_1608Metric_Pad1.08x0.95mm_HandSolder")
-    )
     (path "/15ecaf05-f669-4079-8d71-95c8f3ff2102"
