File: mp3/mp3.kicad_sch (KiCad schematic)
At the start: 33 parts, among them J1 USB4105-GF-A, J2 LEFT, J3 DEBUG, J4 RIGHT, U1 W25Q128JV, U2 RP2040, U3 MCP1702T-3302E_CB, Y1 12MHz

Commit message: second revision of rp devboard
Connections:
- net GND: no longer Y1.2
- net at Y1.1: no longer U2.20 (XIN)
- net at Y1.3: no longer U2.21 (XOUT)
Other:
- moved on the sheet: Y1
Changed lines of the file:
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@@
     (pin "1")
   )
-  (symbol (lib_id "Eclectronics:Crystal") (at 74.93 64.77 270) (unit 1)
+  (symbol (lib_id "Eclectronics:Crystal") (at 74.93 64.77 180) (unit 1)
     (in_bom yes) (on_board yes)
-    (property "Reference" "Y1" (id 0) (at 78.74 63.5 90)
+    (property "Reference" "Y1" (id 0) (at 76.2 68.58 90)
       (effects (font (size 1.27 1.27)) (justify left))
     )
-    (property "Value" "12MHz" (id 1) (at 78.74 66.04 90)
+    (property "Value" "12MHz" (id 1) (at 73.66 68.58 90)
       (effects (font (size 1.27 1.27)) (justify left))
     )
